Commit message: robo_controller hold position

File: ros/src/armvision_description/urdf/armvision.urdf.xacro (robot description, xacro)
@@ -183,5 +183,10 @@
         <limit lower="0.0" upper="${PI/2}" effort="${effort}" velocity="${velocity}" />
     </joint>
-    <!--
+    <link name="end_effector" />
+    <joint name="claw_support_to_end_effector" type="fixed">
+        <parent link="claw_support" />
+        <child link="end_effector" />
+        <origin xyz="-0.09 0.13 -0.1" rpy="0 0 0" />
+    </joint>
     <link name="rgb_camera">
         <xacro:default_inertial mass="0.001" />
@@ -193,18 +198,9 @@
             </geometry>
         </visual>
-        <collision>
-            <origin rpy="-${PI/2} 0 0" xyz="-0.125 0 0.34" />
-            <geometry>
-                <mesh filename="package://armvision_description/meshes/pi_camera.STL"
-                    scale="0.01 0.01 0.01" />
-            </geometry>
-        </collision>
-    </link> -->
-    <!-- <joint name='claw-to-camera' type="fixed">
-        <origin rpy="0 0 0" xyz=" 0 -0.1 0.05" />
+    </link>
+    <joint name="claw_to_camera" type="fixed">
         <parent link="claw_support" />
         <child link="rgb_camera" />
-        <axis xyz='0 0 1' />
-        <limit lower="-${PI/2}" upper="${PI/2}" effort="${effort}" velocity="${velocity}" />
-    </joint> -->
+        <origin xyz="0 -0.1 0.05" rpy="0 0 0" />
+    </joint>
 </robot>

Commit message: final executor and controller fixes

File: ros/src/armvision_description/urdf/armvision.urdf.xacro (robot description, xacro)
@@ -1,6 +1,6 @@
 <?xml version='1.0'?>
 <robot xmlns:xacro="http://www.ros.org/wiki/xacro" name="armvision">
-    <xacro:arg name="is_ignition" default="true" />
-    <xacro:include filename="$(find armvision_description)/urdf/armvision_gazebo.xacro" />
+    <!-- <xacro:arg name="is_ignition" default="true" /> -->
+    <!-- <xacro:include filename="$(find armvision_description)/urdf/armvision_gazebo.xacro" /> -->
     <!-- <xacro:include filename="$(find armvision_description)/urdf/sensors.xacro" /> -->
     <xacro:include filename="$(find armvision_description)/urdf/armvision_ros2_control.xacro" />
@@ -168,18 +168,18 @@
         </collision>
     </link>
-    <joint name="joint_4" type="revolute">
+    <joint name="joint_4" type="fixed">
         <parent link="claw_support" />
         <child link="gripper_right" />
         <axis xyz="0 0 1" />
         <origin rpy="0 0 0" xyz="0.04 0.13 -0.1" />
-        <limit lower="-${PI/2}" upper="0.0" effort="${effort}" velocity="${velocity}" />
-    </joint>
-    <joint name="joint_5" type="revolute">
+        <!-- <limit lower="-${PI/2}" upper="0.0" effort="${effort}" velocity="${velocity}" /> -->
+    </joint>
+    <joint name="joint_5" type="fixed">
         <parent link="claw_support" />
         <child link="gripper_left" />
         <axis xyz="0 0 1" />
         <origin rpy="0 0 0" xyz="-0.22 0.13 -0.1" />
-        <mimic joint="joint_4" multiplier="-1" />
-        <limit lower="0.0" upper="${PI/2}" effort="${effort}" velocity="${velocity}" />
+        <!-- <mimic joint="joint_4" multiplier="-1" />
+        <limit lower="0.0" upper="${PI/2}" effort="${effort}" velocity="${velocity}" /> -->
     </joint>
     <link name="end_effector" />

Commit message: ros2 isaac integration rework

File: ros/src/armvision_description/urdf/armvision.urdf.xacro (robot description, xacro)
@@ -1,6 +1,4 @@
 <?xml version='1.0'?>
 <robot xmlns:xacro="http://www.ros.org/wiki/xacro" name="armvision">
-    <!-- <xacro:arg name="is_ignition" default="true" /> -->
-    <!-- <xacro:include filename="$(find armvision_description)/urdf/armvision_gazebo.xacro" /> -->
     <!-- <xacro:include filename="$(find armvision_description)/urdf/sensors.xacro" /> -->
     <xacro:include filename="$(find armvision_description)/urdf/armvision_ros2_control.xacro" />
@@ -8,10 +6,12 @@
     <xacro:property name="effort" value="30.0" />
     <xacro:property name="velocity" value="10.0" />
-    <xacro:macro name="default_inertial" params="mass">
+    <!-- Solid box approximation: x y z are the box dimensions, com is the center of mass -->
+    <xacro:macro name="box_inertial" params="mass x y z com">
         <inertial>
+            <origin rpy="0 0 0" xyz="${com}" />
             <mass value="${mass}" />
-            <inertia ixx="1.0" ixy="0.0" ixz="0.0"
-                iyy="1.0" iyz="0.0"
-                izz="1.0"
+            <inertia ixx="${mass / 12.0 * (y*y + z*z)}" ixy="0.0" ixz="0.0"
+                iyy="${mass / 12.0 * (x*x + z*z)}" iyz="0.0"
+                izz="${mass / 12.0 * (x*x + y*y)}"
             />
         </inertial>
@@ -19,5 +19,5 @@
     <link name="world" />
     <link name="base_link">
-        <xacro:default_inertial mass="1.0" />
+        <xacro:box_inertial mass="1.0" x="0.3" y="0.3" z="0.3" com="0 0 0.15" />
         <visual>
             <origin rpy="0 0 0" xyz="-0.5 -0.5 0" />
@@ -41,5 +41,5 @@
     </joint>
     <link name="base_plate">
-        <xacro:default_inertial mass="0.1" />
+        <xacro:box_inertial mass="0.1" x="0.2" y="0.2" z="0.35" com="0 0 0.175" />
         <visual>
             <origin rpy="0 0 0" xyz="-0.39 -0.39 -0.56" />
@@ -65,5 +65,5 @@
     </joint>
     <link name="forward_drive_arm">
-        <xacro:default_inertial mass="0.1" />
+        <xacro:box_inertial mass="0.1" x="0.05" y="0.05" z="0.8" com="0 0 0.4" />
         <visual>
             <origin rpy="0 -${PI/2} ${PI/2}" xyz="0.19 0.06 -0.08" />
@@ -89,5 +89,5 @@
     </joint>
     <link name="horizontal_arm">
-        <xacro:default_inertial mass="0.1" />
+        <xacro:box_inertial mass="0.1" x="0.05" y="0.82" z="0.05" com="0 0.41 0" />
         <visual>
             <origin rpy="${PI/2} 0 ${PI/2}" xyz="-0.03 -0.4 -0.06" />
@@ -113,5 +113,5 @@
     </joint>
     <link name="claw_support">
-        <xacro:default_inertial mass="0.05" />
+        <xacro:box_inertial mass="0.05" x="0.1" y="0.1" z="0.1" com="0 0 0" />
         <visual>
             <origin rpy="0 0 ${PI/2}" xyz="0 -0.05 -0.15" />
@@ -135,5 +135,5 @@
     </joint>
     <link name="gripper_right">
-        <xacro:default_inertial mass="0.01" />
+        <xacro:box_inertial mass="0.01" x="0.02" y="0.1" z="0.02" com="0 0 0" />
         <visual>
             <origin rpy="0 0 -${PI/2}" xyz="-0.1 0.5 -0.1" />
@@ -152,5 +152,5 @@
     </link>
     <link name="gripper_left">
-        <xacro:default_inertial mass="0.01" />
+        <xacro:box_inertial mass="0.01" x="0.02" y="0.1" z="0.02" com="0 0 0" />
         <visual>
             <origin rpy="0 0 -${PI/2}" xyz="-0.04 0.5 -0.1" />
@@ -190,5 +190,5 @@
     </joint>
     <link name="rgb_camera">
-        <xacro:default_inertial mass="0.001" />
+        <xacro:box_inertial mass="0.001" x="0.03" y="0.03" z="0.03" com="0 0 0" />
         <visual>
             <origin rpy="-${PI/2} 0 0" xyz="-0.125 0 0.34" />
