Commit message: isaac sim scripting, camera triangulation

File: ros/src/armvision_description/urdf/armvision.urdf (robot description, URDF)
Before this commit: robot armvision, 10 links, 9 joints
Links:
- added link left_camera
- added link right_camera
Joints:
- removed joint claw_to_camera
- added joint plate_to_camera: type fixed, parent base_plate, child rgb_camera, origin xyz=0 0.45 0.2 rpy=0 -0.5 1.57
- added joint rgb_to_left_camera: type fixed, parent rgb_camera, child left_camera, origin xyz=-0.03 0 0 rpy=0 0 0
- added joint rgb_to_right_camera: type fixed, parent rgb_camera, child right_camera, origin xyz=0.03 0 0 rpy=0 0 0

File: ros/src/armvision_description/urdf/armvision.urdf.xacro (robot description, xacro)
@@ -193,5 +193,5 @@
         <xacro:box_inertial mass="0.001" x="0.03" y="0.03" z="0.03" com="0 0 0" />
         <visual>
-            <origin rpy="-${PI/2} 0 0" xyz="-0.125 0 0.34" />
+            <origin rpy="-1.57 0 -1.57" xyz="-0.1 0.125 0.15" />
             <geometry>
                 <mesh filename="package://armvision_description/meshes/pi_camera.STL"
@@ -200,8 +200,20 @@
         </visual>
     </link>
-    <joint name="claw_to_camera" type="fixed">
-        <parent link="claw_support" />
+    <joint name="plate_to_camera" type="fixed">
+        <parent link="base_plate" />
         <child link="rgb_camera" />
-        <origin xyz="0 -0.1 0.05" rpy="0 0 0" />
+        <origin xyz="0 0.45 0.2" rpy="0 -0.5 1.57" />
+    </joint>
+    <link name="left_camera" />
+    <joint name="rgb_to_left_camera" type="fixed">
+        <parent link="rgb_camera" />
+        <child link="left_camera" />
+        <origin xyz="-0.03 0 0" rpy="0 0 0" />
+    </joint>
+    <link name="right_camera" />
+    <joint name="rgb_to_right_camera" type="fixed">
+        <parent link="rgb_camera" />
+        <child link="right_camera" />
+        <origin xyz="0.03 0 0" rpy="0 0 0" />
     </joint>
 </robot>
